File: kvio_core.kicad_pcb (KiCad board)
At the start: 6 copper layers, 98 x 30 mm, 288 parts, among them J1001 12-pin_FFC_(SFV12R), J1301 USB3_B_Micro, J301 Conn_01x06_Male, J401 12-pin_FFC_(SFV12R), J801 12-pin_FFC_(SFV12R), J901 12-pin_FFC_(SFV12R), Q1201 NTZD3155C, U1001 IP4254CZ8-4-TTL, U1002 EMI8143, U101 xc7a100t-csg324, U1101 AR0135CS, U1201 MT41J128M16JT-125:K, U1202 ASM330LHH, U1301 FT601Q, U1302 EMI8143, U1401 AR0135CS, U201 FAN53541, U202 FAN53541, U203 FAN53541, U204 FAN53541, U301 MX25L6433F, U302 MAX809, U401 EMI8143, U402 IP4254CZ8-4-TTL, U801 IP4254CZ8-4-TTL, U802 EMI8143, U901 IP4254CZ8-4-TTL, U902 EMI8143, Y1301 Crystal_GND24_Small

Commit message: More work
Parts:
- removed J301: Conn_01x06_Male, Connector_PinSocket_1.27mm:PinSocket_2x03_P1.27mm_Vertical
- removed R317, R318, R319, R320: 100, passive:R_0402
- added C101: 0.1u, passive:C_0201, F.Cu at (202.7, 113.2)
- added R101: 10k, passive:R_0402, F.Cu at (198.5, 112.9)
- added U102: 100 MHz, crystals:Crystal_SMD_2520-4Pin_2.5x2.0mm, F.Cu at (200.6, 112.9)
- added U303: IP4254CZ8-4-TTL, dfn:UDFN-8-1EP_1.7x1.35mm_P0.4mm_EP0.4x1.2mm, B.Cu at (211.8, 113.1)
- added U304: SOICbite_JTAG, connectors:SOICbiteSmall, F.Cu at (218.2, 114.6)
- C1104, R1401, R1403, R1404: moved to B.Cu
- Y1301: footprint Crystal:Crystal_SMD_2520-4Pin_2.5x2.0mm -> crystals:Crystal_SMD_2520-4Pin_2.5x2.0mm
- moved R1213 54.3 mm to (178.8, 93.0)
- moved R1214 54.3 mm to (179.2, 94.5)
- moved R1215 54.3 mm to (181.5, 91.2)
- moved R1210 54.1 mm to (173.2, 91.8)
- moved R1217 49.9 mm to (174.0, 93.6), turned to 180 degrees
- moved R1216 47.4 mm to (174.4, 96.6), turned to 90 degrees
- moved C1414 31.0 mm to (240.0, 99.5), turned to 180 degrees
- moved RN1102 28.3 mm to (231.0, 106.9), turned to 180 degrees
- moved RN1103 28.3 mm to (231.0, 104.4), turned to 180 degrees
- moved C1413 28.0 mm to (240.0, 101.5), turned to 180 degrees
- moved RN1104 27.7 mm to (231.4, 95.9), turned to 90 degrees
- moved C1410 27.0 mm to (238.0, 103.1), turned to 180 degrees
- moved C1405 26.9 mm to (238.0, 100.0), turned to 180 degrees
- moved C1411 26.8 mm to (238.0, 98.5), turned to 180 degrees
- moved C1406 25.5 mm to (238.0, 101.5), turned to 180 degrees
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Connections:
- R1210 pad 1: /Sensors/IMU_INT_P -> /IMU_INT
Routing:
- net GND: track 215.8 -> 233.2 mm, vias 135 -> 147
- net /Config/TDI_P: track 0.00 -> 9.78 mm
- net /sheet5D568411/D0_P: track 11.4 -> 2.25 mm
- net /Config/TCK_P: track 0.00 -> 8.51 mm
- net /sheet5D568411/D4_P: track 10.8 -> 2.68 mm
- net /USB3 Interface/GLCLK_100MHZ: track 5.40 -> 13.0 mm, vias 1 -> 2
- net /Config/TDO_P: track 0.00 -> 7.26 mm
- net /sheet5D568411/D1_P: track 10.1 -> 3.48 mm
- net +3V3: track 40.5 -> 46.5 mm, vias 27 -> 29
- net /Config/TMS_P: track 0.00 -> 5.98 mm
- net /sheet5D568411/D5_P: track 9.58 -> 3.78 mm
- net /sheet5D568411/D11_P: track 7.85 -> 12.8 mm
- net VAA: track 16.4 -> 20.9 mm
- net /sheet5D568411/D2_P: track 8.93 -> 4.68 mm
- net /sheet5D568411/D6_P: track 8.37 -> 4.74 mm
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Other:
- outline, holes or cut-outs redrawn
- board text added: "JTAG"

Commit message: More layout
Parts:
- removed H104: MountingHole_Pad, MountingHole:MountingHole_2.2mm_M2_Pad_Via
- moved H102 26.8 mm to (231.0, 90.0)
- moved C1201 23.0 mm to (222.1, 97.4), turned to 270 degrees
- moved R1201 22.0 mm to (222.9, 97.2), turned to 270 degrees
- moved C236 21.5 mm to (214.2, 93.5), turned to 90 degrees
- moved R1202 21.2 mm to (222.9, 98.9), turned to 270 degrees
- moved C1202 20.5 mm to (222.1, 98.7), turned to 270 degrees
- moved C252 19.9 mm to (211.0, 96.6), turned to 270 degrees
- moved C284 18.3 mm to (210.2, 98.2), turned to 270 degrees
- moved C244 18.2 mm to (212.6, 95.8), turned to 90 degrees
- moved C224 18.0 mm to (212.6, 99.8), turned to 270 degrees
- moved C230 16.8 mm to (208.6, 95.8), turned to 270 degrees
- moved U801 3.98 mm to (188.1, 27.4)
- moved C1211 1.44 mm to (224.7, 100.6), turned to 90 degrees
- moved C1215 1.17 mm to (225.6, 98.6)
Routing:
- net /USB3 Interface/VBUS: track 0.00 -> 18.7 mm
- net /DDR Memory/VREF: track 3.94 -> 14.2 mm
- net GND: track 233.2 -> 239.1 mm, vias 147 -> 149
- net +3V3: track 46.5 -> 49.7 mm
- net /DDR Memory/DDR3_VDD: track 26.5 -> 29.0 mm, vias 17 -> 18
- net /CAM1_PIXCLK: track 0.00 -> 0.62 mm, vias 0 -> 1
- net /CAM1_LV: track 0.00 -> 0.62 mm, vias 0 -> 1
- net /CAM1_D8: track 0.00 -> 0.62 mm, vias 0 -> 1
- net /CAM1_D10: track 0.00 -> 0.62 mm, vias 0 -> 1
- net /CAM1_D5: track 0.00 -> 0.62 mm, vias 0 -> 1
- net /CAM1_D1: track 0.00 -> 0.62 mm, vias 0 -> 1
- net /CAM1_FV: track 0.00 -> 0.62 mm, vias 0 -> 1
- net /CAM1_FLASH: track 0.00 -> 0.62 mm, vias 0 -> 1
- net /CAM1_D9: track 0.00 -> 0.62 mm, vias 0 -> 1
- net /CAM1_D7: track 0.00 -> 0.62 mm, vias 0 -> 1
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Other:
- net class Default: clearance 0.0889 -> 0.1
- net class power: clearance 0.0889 -> 0.1
- rule trace_clearance: 0.0889 -> 0.1
- board text added: "By Emil Fresk, 2019"

Commit message: More layout
Parts:
- moved C233 0.10 mm to (202.1, 104.6)
Routing:
- net /CAM0_D8: track 0.62 -> 28.2 mm
- net /CAM0_D9: track 0.62 -> 27.9 mm
- net /CAM0_D10: track 0.62 -> 27.6 mm
- net /CAM1_D3: track 0.62 -> 27.3 mm
- net /CAM0_D11: track 0.62 -> 27.3 mm
- net /CAM1_D2: track 0.62 -> 27.0 mm
- net /CAM0_LV: track 0.62 -> 26.7 mm
- net /CAM1_D1: track 0.62 -> 26.7 mm
- net /CAM0_FV: track 0.62 -> 26.4 mm
- net /CAM1_D0: track 0.62 -> 26.4 mm
- net /CAM0_PIXCLK: track 0.62 -> 26.1 mm
- net /CAM1_D7: track 0.62 -> 25.8 mm
- net /CAM0_FLASH: track 0.62 -> 25.8 mm
- net /CAM1_D6: track 0.62 -> 25.5 mm
- net /CAM1_D5: track 0.62 -> 25.2 mm
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Other:
- outline, holes or cut-outs redrawn
